File: mt-rt.kicad_pcb (KiCad board)
At the start: 2 copper layers, 0 parts

Commit message: Added Rotary Encoder with switch
Added Custom Part Library
Added Encoder to Library
Parts:
- added SW1: RotaryEncoder_Switch_4P, Custom_Parts:Rotary_Switch_4P, F.Cu at (42.5, 53.8)
Other:
- board outline added: 3 x 2.1 mm
