File: HMI.kicad_sch (KiCad schematic)
At the start: 5 parts, among them SW1 RotaryEncoder_Switch_4P

Commit message: annotated full sheet
Parts:
- gave numbers to parts that had none: 2
- renumbered SW2 to SW3, SW3 to SW4
Changed lines of the file:
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@@
 		(dnp no)
 		(fields_autoplaced yes)
-		(property "Reference" "LCD?"
+		(property "Reference" "LCD1"
 			(at 231.14 55.8799 0)
 			(effects
@@
 			(project ""
 				(path "/ee47f507-02e8-4ef5-a6d4-1ac4b2022b93/1ab1902b-acf7-4c4c-8c09-61d5cb12072a"
-					(reference "LCD?")
+					(reference "LCD1")
 					(unit 1)
 				)
@@
 		(dnp no)
 		(fields_autoplaced yes)
-		(property "Reference" "SW?"
+		(property "Reference" "SW2"
 			(at 69.85 93.3449 0)
 			(effects
@@
 			(project ""
 				(path "/ee47f507-02e8-4ef5-a6d4-1ac4b2022b93/1ab1902b-acf7-4c4c-8c09-61d5cb12072a"
-					(reference "SW?")
+					(reference "SW2")
 					(unit 1)
 				)
@@
 		(dnp no)
 		(fields_autoplaced yes)
-		(property "Reference" "SW2"
+		(property "Reference" "SW3"
 			(at 71.12 121.2849 0)
 			(effects
@@
 			(project "mt-rt"
 				(path "/ee47f507-02e8-4ef5-a6d4-1ac4b2022b93/1ab1902b-acf7-4c4c-8c09-61d5cb12072a"
-					(reference "SW2")
+					(reference "SW3")
 					(unit 1)
 				)
@@
 		(dnp no)
 		(fields_autoplaced yes)
-		(property "Reference" "SW3"
+		(property "Reference" "SW4"
 			(at 71.12 147.9549 0)
 			(effects
@@
 			(project "mt-rt"
 				(path "/ee47f507-02e8-4ef5-a6d4-1ac4b2022b93/1ab1902b-acf7-4c4c-8c09-61d5cb12072a"
-					(reference "SW3")
+					(reference "SW4")
 					(unit 1)
 				)
