File: sensors_and_drivers.kicad_sch (KiCad schematic)
At the start: 1 part

Commit message: annotated full sheet
Parts:
- gave numbers to parts that had none: 1
Changed lines of the file:
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@@
 		(dnp no)
 		(fields_autoplaced yes)
-		(property "Reference" "U?"
+		(property "Reference" "U2"
 			(at 68.58 40.64 0)
 			(effects
@@
 			(project ""
 				(path "/ee47f507-02e8-4ef5-a6d4-1ac4b2022b93/89e6ea21-7a60-4e98-9e90-22537fd40aae"
-					(reference "U?")
+					(reference "U2")
 					(unit 1)
 				)
